File: hardware/flight_controller_v1/main_pcb/main_pcb.kicad_sch (KiCad schematic)
At the start: 19 parts, among them U5 L78L33_SOT89, U7 NEO-M8N

Commit message: Slight changes to PCB
Parts:
- C1: value (none) -> 0.1uF; footprint (none) -> Capacitor_SMD:C_0805_2012Metric
- C11: value (none) -> 10uF
- C12: value (none) -> 0.1uF
- C2: value (none) -> 10uF; footprint (none) -> Capacitor_SMD:CP_Elec_5x3
- M1, M2, M3, M4: value (none) -> Conn_01x03; footprint (none) -> Connector_PinHeader_2.54mm:PinHeader_1x03_P2.54mm_Horizontal
- U1: value (none) -> CH340E; footprint (none) -> Package_SO:MSOP-10_3x3mm_P0.5mm
- U2: value (none) -> ICM-20948; footprint (none) -> Sensor_Motion:InvenSense_QFN-24_3x3mm_P0.4mm
- U3: value (none) -> TLV70018_SOT23-5; footprint (none) -> Package_TO_SOT_SMD:SOT-23-5
- U8: value (none) -> ESP32-WROOM-32U; footprint (none) -> RF_Module:ESP32-WROOM-32U
- bat_power1: value (none) -> Conn_01x02; footprint (none) -> Connector_PinHeader_2.54mm:PinHeader_1x02_P2.54mm_Horizontal
Connections:
- net +3V3: now also U2.13 (VDD), U3.1 (IN)
- net GND: now also U2.18 (GND), U2.20 (GND), U3.2 (GND)
- net MPU_INT: now reaches U2.12 (INT1)
- net +1V8: now reaches U2.8 (VDDIO)
- net +1V8: now also U3.5 (OUT)

Commit message: New PCB iteration
Parts:
- removed L1: L, symbol Device:L
- removed U1: CH340E, Package_SO:MSOP-10_3x3mm_P0.5mm, symbol Interface_USB:CH340E
- removed U2: ICM-20948, Sensor_Motion:InvenSense_QFN-24_3x3mm_P0.4mm, symbol Sensor_Motion:ICM-20948
- removed U3: TLV70018_SOT23-5, Package_TO_SOT_SMD:SOT-23-5, symbol Regulator_Linear:TLV70018_SOT23-5
- removed UART_DWNLD1: Conn_01x03, Connector_PinHeader_2.54mm:PinHeader_1x03_P2.54mm_Horizontal, symbol Connector_Generic:Conn_01x03
- added C3, C8: 4.7uF, Capacitor_SMD:C_0805_2012Metric, symbol Device:C
- added C4, C5, C7, C9: 0.1uF, Capacitor_SMD:C_0805_2012Metric, symbol Device:C
- added C6: 1uF, Capacitor_SMD:C_0805_2012Metric, symbol Device:C
- added EEPROM1: 24LC32, Package_SO:TSSOP-8_4.4x3mm_P0.65mm, symbol Memory_EEPROM:24LC32
- added J1: Conn_01x06, Connector_PinHeader_2.54mm:PinHeader_1x06_P2.54mm_Vertical, symbol Connector_Generic:Conn_01x06
- added J2: Conn_01x04_Female, Connector_PinHeader_2.54mm:PinHeader_1x04_P2.54mm_Vertical, symbol Connector:Conn_01x04_Female
- added J3: (no value), symbol Connector_Generic:Conn_02x06_Counter_Clockwise
- added J4: (no value), symbol Connector_Generic:Conn_02x03_Odd_Even
- added R1: 22.1k, Resistor_SMD:R_0805_2012Metric, symbol Device:R
- added R2: 47.5k, Resistor_SMD:R_0805_2012Metric, symbol Device:R
- added R4, R5: 10k, Resistor_SMD:R_0805_2012Metric, symbol Device:R
- added R6: 3M, Resistor_SMD:R_0805_2012Metric, symbol Device:R
- added R7: 1M, Resistor_SMD:R_0805_2012Metric, symbol Device:R
- added SW1: SW_Push, Button_Switch_SMD:SW_SPST_B3U-1000P-B, symbol Switch:SW_Push
- added U1: L78L33_SOT89, Package_TO_SOT_SMD:SOT-89-3, symbol Regulator_Linear:L78L33_SOT89
- added U2: LM2904, Package_SO:Diodes_PSOP-8, symbol Amplifier_Operational:LM2904
- added U6: CP2102N-Axx-xQFN20, Package_DFN_QFN:MLF-20-1EP_4x4mm_P0.5mm_EP2.6x2.6mm, symbol Interface_USB:CP2102N-Axx-xQFN20
- added U9: LSM6DS3, Package_LGA:LGA-14_3x2.5mm_P0.5mm_LayoutBorder3x4y, symbol Sensor_Motion:LSM6DS3
- BAT1: renamed from bat_power1; footprint Connector_PinHeader_2.54mm:PinHeader_1x02_P2.54mm_Horizontal -> Connector_PinHeader_2.54mm:PinHeader_1x02_P2.54mm_Vertical
- C10: value 10nF -> 0.1uF; footprint (none) -> Capacitor_SMD:C_0805_2012Metric
- C11, C12: footprint (none) -> Capacitor_SMD:C_0805_2012Metric
- C2: footprint Capacitor_SMD:CP_Elec_5x3 -> Capacitor_SMD:CP_Elec_5x4.5
- M1, M2, M3, M4: footprint Connector_PinHeader_2.54mm:PinHeader_1x03_P2.54mm_Horizontal -> Connector_PinHeader_2.54mm:PinHeader_1x03_P2.54mm_Vertical
- R3: value R -> 10k; footprint (none) -> Resistor_SMD:R_0805_2012Metric
- renumbered U8 to ESP32-WROOM-32U1, U7 to GPS1
Connections:
- net +3V3: now also C10.1, GPS1.22 (V_BCKP), GPS1.23 (VCC), R3.2, C5.1, C7.2, C8.1, C9.1, EEPROM1.8 (VCC), J1.5 (Pin_5), J2.4 (Pin_4), J3.2 (Pin_2), U1.1 (OUT), U6.6 (VDD), U9.5 (VDDIO), U9.8 (VDD)
- net GND: now also C10.2, GPS1.10 (GND), GPS1.12 (GND), GPS1.13 (GND), GPS1.24 (GND), C3.1, C4.1, C5.2, C6.1, C7.1, C8.2, C9.2, EEPROM1.1 (A0), EEPROM1.2 (A1), EEPROM1.3 (A2), EEPROM1.4 (GND), EEPROM1.7 (WP), J1.4 (Pin_4), J2.1 (Pin_1), J3.1 (Pin_1), R2.2, R4.2, R5.2, R7.2, SW1.1, U1.2 (GND), U2.4 (V-), U6.12 (GND), U6.21 (GND), U6.3 (GND), U9.6 (GND), U9.7 (GND)
- net M1: now also ESP32-WROOM-32U1.7 (IO35)
- net M2: now also ESP32-WROOM-32U1.26 (IO4)
- net M3: now also ESP32-WROOM-32U1.31 (IO19)
- net M4: now also ESP32-WROOM-32U1.14 (IO12)
- net RX: now also J1.3 (Pin_3), U6.18 (TXD)
- net TX: now also J1.2 (Pin_2), U6.17 (RXD)
- net USB+: now also J4.3 (Pin_3)
- net USB-: now also J4.4 (Pin_4)
- net v_bat: now also R6.1, U2.8 (V+)
- net RESET: now reaches R3.1
- net RESET: now also ESP32-WROOM-32U1.3 (EN), GPS1.8 (~{RESET}), C6.2, J1.1 (Pin_1), SW1.2, U6.9 (~{RST})
- net gps_antenna: now reaches GPS1.11 (RF_IN)
- net SDA_eeprom: now reaches GPS1.18 (SDA/~{SPI_CS})
- net SDA_eeprom: now also EEPROM1.5 (SDA)
- net SCL_eeprom: now reaches GPS1.19 (SCL/SPI_CLK)
- net SCL_eeprom: now also EEPROM1.6 (SCL)
- net GPS_TX: now reaches GPS1.20 (TXD/SPI_MISO)
- net GPS_TX: now also ESP32-WROOM-32U1.9 (IO33)
- net GPS_RX: now reaches GPS1.21 (RXD/SPI_MOSI)
- net GPS_RX: now also ESP32-WROOM-32U1.8 (IO32)
- net USB-gps: now reaches GPS1.5 (USB_DM)
- net USB-gps: now also J4.2 (Pin_2)
- net USB+gps: now reaches GPS1.6 (USB_DP)
- net USB+gps: now also J4.1 (Pin_1)
- net xIO3: now reaches ESP32-WROOM-32U1.10 (IO25)
- net xIO3: now also J3.10 (Pin_10)
- net xIO2: now reaches ESP32-WROOM-32U1.11 (IO26)
- net xIO2: now also J3.8 (Pin_8)
- net xIO1: now reaches ESP32-WROOM-32U1.12 (IO27)
- net xIO1: now also J3.6 (Pin_6)
- net xIO6: now reaches ESP32-WROOM-32U1.13 (IO14)
- net xIO6: now also ESP32-WROOM-32U1.6 (IO34), J3.4 (Pin_4)
- net xIO4: now reaches ESP32-WROOM-32U1.16 (IO13)
- net xIO4: now also J3.5 (Pin_5)
- net xIO5: now reaches ESP32-WROOM-32U1.23 (IO15)
- net xIO5: now also J3.3 (Pin_3)
- net VBAT_LL: now reaches ESP32-WROOM-32U1.24 (IO2)
- net VBAT_LL: now also U2.1, U2.2 (-)
- net xIO7: now reaches ESP32-WROOM-32U1.27 (IO16)
- net xIO7: now also J3.7 (Pin_7)
- net xIO8: now reaches ESP32-WROOM-32U1.28 (IO17)
- net xIO8: now also J3.9 (Pin_9)
- net xIO10: now reaches ESP32-WROOM-32U1.29 (IO5)
- net xIO10: now also J3.11 (Pin_11)
- net xIO9: now reaches ESP32-WROOM-32U1.30 (IO18)
- net xIO9: now also J3.12 (Pin_12)
- net SDA: now reaches ESP32-WROOM-32U1.33 (IO21)
- net SDA: now also J2.2 (Pin_2), R4.1, U9.14 (SDA)
- net SCL: now reaches ESP32-WROOM-32U1.36 (IO22)
- net SCL: now also J2.3 (Pin_3), R5.1, U9.13 (SCL)
- net MPU_INT_1: now reaches ESP32-WROOM-32U1.37 (IO23)
- net MPU_INT_1: now also U9.4 (INT1)
- new net: R1.2, R2.1, U6.8 (VBUS)
- new net: R6.2, R7.1, U2.3 (+)
- new net AUX_CL: U9.3 (SCX)
- new net AUX_DA: U9.2 (SDX)
- new net MPU_INT_2: U9.9 (INT2)
- new net USB+prog: J4.5 (Pin_5), U6.4 (D+)
- new net USB-prog: J4.6 (Pin_6), U6.5 (D-)
- new net USB5V: C3.2, C4.2, J1.6 (Pin_6), R1.1, U1.3 (IN), U6.7 (VREGIN)
Other:
- note added: "Reset"
- note added: "USB interface"
- note added: "USB-switcher"
- note added: "Voltage detect"

Commit message: Code restructuring in progress..
Parts:
- J3: value (none) -> Conn_02x06_Counter_Clockwise; footprint (none) -> Connector_PinHeader_2.54mm:PinHeader_2x06_P2.54mm_Vertical
- J4: value (none) -> Conn_02x03_Odd_Even; footprint (none) -> Connector_PinHeader_2.54mm:PinHeader_2x03_P2.54mm_Vertical
Changed lines of the file:
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@@
     (in_bom yes) (on_board yes) (fields_autoplaced)
     (property "Reference" "J3" (id 0) (at 171.45 67.31 0))
-    (property "Value" "" (id 1) (at 171.45 69.85 0))
-    (property "Footprint" "" (id 2) (at 170.18 78.74 0)
+    (property "Value" "Conn_02x06_Counter_Clockwise" (id 1) (at 171.45 69.85 0))
+    (property "Footprint" "Connector_PinHeader_2.54mm:PinHeader_2x06_P2.54mm_Vertical" (id 2) (at 170.18 78.74 0)
       (effects (font (size 1.27 1.27)) hide)
     )
@@
     (in_bom yes) (on_board yes) (fields_autoplaced)
     (property "Reference" "J4" (id 0) (at 144.78 161.29 0))
-    (property "Value" "" (id 1) (at 144.78 163.83 0))
-    (property "Footprint" "" (id 2) (at 143.51 170.18 0)
-      (effects (font (size 1.27 1.27)) hide)
-    )
+    (property "Value" "Conn_02x03_Odd_Even" (id 1) (at 144.78 163.83 0))
+    (property "Footprint" "Connector_PinHeader_2.54mm:PinHeader_2x03_P2.54mm_Vertical" (id 2) (at 143.51 170.18 0)
+      (effects (font (size 1.27 1.27)) hide)
+    )
